Commit message: udpates

File: src/mks_description/urdf/diffbot.urdf (robot description, URDF)
Before this commit: robot diffbot, 2 links, 1 joints
Links:
- link base_link: mass 5 -> 10; geometry collision box size=1.0 1.0 1.0; visual box size=1.0 1.0 1.0
Joints:
- joint world_to_base: origin xyz=0 0 0 rpy=0 0 0 -> xyz=0 0 5 rpy=0 0 0
