Commit message: legs working

File: src/mks_description/urdf/eve.urdf.xacro (robot description, xacro)
@@ -10,5 +10,5 @@
         </visual>
         <collision>
-            <origin xyz="0 0 0" rrpy="${pi/2} 0 0"/>
+            <origin xyz="0 0 0" rpy="${pi/2} 0 0"/>
             <geometry>
                 <mesh filename="package://mks_description/meshes/chassis.stl" scale="0.001 0.001 0.001"/>
@@ -28,5 +28,5 @@
     <link name="front_left_leg">
         <visual>
-            <origin xyz="$(eval -0.245) $(eval 0.056899) $(eval -0.024317)" rpy="${pi/2} 0 0"/>
+            <origin xyz="-0.247 0.058093 -0.025691" rpy="${pi/2} 0 0"/>
             <geometry>
                 <mesh filename="package://mks_description/meshes/front_left_leg.stl" scale="0.001 0.001 0.001"/>
@@ -34,7 +34,85 @@
         </visual>
         <collision>
-            <origin xyz="0 0 0" rpy="${pi/2} 0 0"/>
+            <origin xyz="-0.247 0.058093 -0.025691" rpy="${pi/2} 0 0"/>
             <geometry>
                 <mesh filename="package://mks_description/meshes/front_left_leg.stl" scale="0.001 0.001 0.001"/>
+            </geometry>
+        </collision>
+        <inertial>
+            <origin xyz="0 0 0" rpy="0 0 0"/>
+            <mass value="5.0"/>
+            <inertia ixx="0.2" ixy="0" ixz="0" iyy="0.3" iyz="0" izz="0.1"/>
+        </inertial>
+    </link>
+    <link name="front_right_leg">
+        <visual>
+            <origin xyz="0.247 0.058093 -0.025691" rpy="${pi/2} 0 0"/>
+            <geometry>
+                <mesh filename="package://mks_description/meshes/front_right_leg.stl" scale="0.001 0.001 0.001"/>
+            </geometry>
+        </visual>
+        <collision>
+            <origin xyz="0.247 0.058093 -0.025691" rpy="${pi/2} 0 0"/>
+            <geometry>
+                <mesh filename="package://mks_description/meshes/front_right_leg.stl" scale="0.001 0.001 0.001"/>
+            </geometry>
+        </collision>
+        <inertial>
+            <origin xyz="0 0 0" rpy="0 0 0"/>
+            <mass value="5.0"/>
+            <inertia ixx="0.2" ixy="0" ixz="0" iyy="0.3" iyz="0" izz="0.1"/>
+        </inertial>
+    </link>
+    <link name="back_left_leg">
+        <visual>
+            <origin xyz="-0.247 -0.058093 -0.025691" rpy="${pi/2} 0 0"/>
+            <geometry>
+                <mesh filename="package://mks_description/meshes/back_left_leg.stl" scale="0.001 0.001 0.001"/>
+            </geometry>
+        </visual>
+        <collision>
+            <origin xyz="-0.247 -0.058093 -0.025691" rpy="${pi/2} 0 0"/>
+            <geometry>
+                <mesh filename="package://mks_description/meshes/back_left_leg.stl" scale="0.001 0.001 0.001"/>
+            </geometry>
+        </collision>
+        <inertial>
+            <origin xyz="0 0 0" rpy="0 0 0"/>
+            <mass value="5.0"/>
+            <inertia ixx="0.2" ixy="0" ixz="0" iyy="0.3" iyz="0" izz="0.1"/>
+        </inertial>
+    </link>
+    <link name="back_right_leg">
+        <visual>
+            <origin xyz="0.247 -0.058093 -0.025691" rpy="${pi/2} 0 0"/>
+            <geometry>
+                <mesh filename="package://mks_description/meshes/back_right_leg.stl" scale="0.001 0.001 0.001"/>
+            </geometry>
+        </visual>
+        <collision>
+            <origin xyz="0.247 -0.058093 -0.025691" rpy="${pi/2} 0 0"/>
+            <geometry>
+                <mesh filename="package://mks_description/meshes/back_right_leg.stl" scale="0.001 0.001 0.001"/>
+            </geometry>
+        </collision>
+        <inertial>
+            <origin xyz="0 0 0" rpy="0 0 0"/>
+            <mass value="5.0"/>
+            <inertia ixx="0.2" ixy="0" ixz="0" iyy="0.3" iyz="0" izz="0.1"/>
+        </inertial>
+    </link>
+    <link name="front_left_wheel">
+        <visual>
+            <origin xyz="-0.3395 0.445977 -0.016173" rpy="${pi/2} 0 0"/>
+            <!-- <origin xyz="0 0 0" rpy="${pi/2} 0 0"/> -->
+            <geometry>
+                <mesh filename="package://mks_description/meshes/front_left_wheel.stl" scale="0.001 0.001 0.001"/>
+            </geometry>
+        </visual>
+        <collision>
+            <origin xyz="-0.3395 0.445977 -0.016173" rpy="${pi/2} 0 0"/>
+            <!-- <origin xyz="0 0 0" rpy="${pi/2} 0 0"/> -->
+            <geometry>
+                <mesh filename="package://mks_description/meshes/front_left_wheel.stl" scale="0.001 0.001 0.001"/>
             </geometry>
         </collision>
@@ -48,8 +126,35 @@
         <parent link="chassis"/>
         <child link="front_left_leg"/>
-        <origin xyz="0 0 0" rpy="0 0 0"/>
-        <origin xyz="0 0 0" rpy="0 0 0"/>
+        <origin xyz="0.247 -0.058093 +0.025691" rpy="0 0 0"/>
         <axis xyz="1 0 0"/>
-        <limit lower="-${0}" upper="${pi}" velocity="1.0" effort="5.0"/>
+        <limit lower="0" upper="${pi/3}" velocity="1.0" effort="5.0"/>
+    </joint>
+    <joint name="front_right_leg_to_chassis" type="revolute">
+        <parent link="chassis"/>
+        <child link="front_right_leg"/>
+        <origin xyz="-0.247 -0.058093 +0.025691" rpy="0 0 0"/>
+        <axis xyz="1 0 0"/>
+        <limit lower="0" upper="${pi/3}" velocity="1.0" effort="5.0"/>
+    </joint>
+    <joint name="back_left_leg_to_chassis" type="revolute">
+        <parent link="chassis"/>
+        <child link="back_left_leg"/>
+        <origin xyz="0.247 0.058093 +0.025691" rpy="0 0 0"/>
+        <axis xyz="1 0 0"/>
+        <limit lower="-${pi/3}" upper="0" velocity="1.0" effort="5.0"/>
+    </joint>
+    <joint name="back_right_leg_to_chassis" type="revolute">
+        <parent link="chassis"/>
+        <child link="back_right_leg"/>
+        <origin xyz="-0.247 0.058093 +0.025691" rpy="0 0 0"/>
+        <axis xyz="1 0 0"/>
+        <limit lower="-${pi/3}" upper="0" velocity="1.0" effort="5.0"/>
+    </joint>
+    <joint name="front_left_wheel_to_leg" type="continuous">
+        <parent link="front_left_leg"/>
+        <child link="front_left_wheel"/>
+        <!-- <origin xyz="0.3395 -0.445977 0.016173" rpy="${pi/2} 0 0"/> -->
+        <origin xyz="0 0 0" rpy="${pi/2} 0 0"/>
+        <axis xyz="1 0 0"/>
     </joint>
 </robot>

Commit message: consistent model

File: src/mks_description/urdf/eve.urdf.xacro (robot description, xacro)
@@ -104,6 +104,5 @@
     <link name="front_left_wheel">
         <visual>
-            <origin xyz="-0.3395 0.445977 -0.016173" rpy="${pi/2} 0 0"/>
-            <!-- <origin xyz="0 0 0" rpy="${pi/2} 0 0"/> -->
+            <origin xyz="-0.3395 0.445997 -0.016173" rpy="${pi/2} 0 0"/>
             <geometry>
                 <mesh filename="package://mks_description/meshes/front_left_wheel.stl" scale="0.001 0.001 0.001"/>
@@ -111,8 +110,64 @@
         </visual>
         <collision>
-            <origin xyz="-0.3395 0.445977 -0.016173" rpy="${pi/2} 0 0"/>
-            <!-- <origin xyz="0 0 0" rpy="${pi/2} 0 0"/> -->
+            <origin xyz="-0.3395 0.445997 -0.016173" rpy="${pi/2} 0 0"/>
             <geometry>
                 <mesh filename="package://mks_description/meshes/front_left_wheel.stl" scale="0.001 0.001 0.001"/>
+            </geometry>
+        </collision>
+        <inertial>
+            <origin xyz="0 0 0" rpy="0 0 0"/>
+            <mass value="5.0"/>
+            <inertia ixx="0.2" ixy="0" ixz="0" iyy="0.3" iyz="0" izz="0.1"/>
+        </inertial>
+    </link>
+    <link name="front_right_wheel">
+        <visual>
+            <origin xyz="0.3395 0.445997 -0.016173" rpy="${pi/2} 0 0"/>
+            <geometry>
+                <mesh filename="package://mks_description/meshes/front_right_wheel.stl" scale="0.001 0.001 0.001"/>
+            </geometry>
+        </visual>
+        <collision>
+            <origin xyz="0.3395 0.445997 -0.016173" rpy="${pi/2} 0 0"/>
+            <geometry>
+                <mesh filename="package://mks_description/meshes/front_right_wheel.stl" scale="0.001 0.001 0.001"/>
+            </geometry>
+        </collision>
+        <inertial>
+            <origin xyz="0 0 0" rpy="0 0 0"/>
+            <mass value="5.0"/>
+            <inertia ixx="0.2" ixy="0" ixz="0" iyy="0.3" iyz="0" izz="0.1"/>
+        </inertial>
+    </link>
+    <link name="back_left_wheel">
+        <visual>
+            <origin xyz="-0.3395 0.445997 -0.016173" rpy="${pi/2} 0 0"/>
+            <geometry>
+                <mesh filename="package://mks_description/meshes/back_left_wheel.stl" scale="0.001 0.001 0.001"/>
+            </geometry>
+        </visual>
+        <collision>
+            <origin xyz="-0.3395 0.445997 -0.016173" rpy="${pi/2} 0 0"/>
+            <geometry>
+                <mesh filename="package://mks_description/meshes/back_left_wheel.stl" scale="0.001 0.001 0.001"/>
+            </geometry>
+        </collision>
+        <inertial>
+            <origin xyz="0 0 0" rpy="0 0 0"/>
+            <mass value="5.0"/>
+            <inertia ixx="0.2" ixy="0" ixz="0" iyy="0.3" iyz="0" izz="0.1"/>
+        </inertial>
+    </link>
+    <link name="back_right_wheel">
+        <visual>
+            <origin xyz="0.3395 0.445997 -0.016173" rpy="${pi/2} 0 0"/>
+            <geometry>
+                <mesh filename="package://mks_description/meshes/back_right_wheel.stl" scale="0.001 0.001 0.001"/>
+            </geometry>
+        </visual>
+        <collision>
+            <origin xyz="0.3395 0.445997 -0.016173" rpy="${pi/2} 0 0"/>
+            <geometry>
+                <mesh filename="package://mks_description/meshes/back_right_wheel.stl" scale="0.001 0.001 0.001"/>
             </geometry>
         </collision>
@@ -154,6 +209,23 @@
         <parent link="front_left_leg"/>
         <child link="front_left_wheel"/>
-        <!-- <origin xyz="0.3395 -0.445977 0.016173" rpy="${pi/2} 0 0"/> -->
-        <origin xyz="0 0 0" rpy="${pi/2} 0 0"/>
+        <origin xyz="0.0925 -0.387904 -0.009518" rpy="0 0 0"/>
+        <axis xyz="1 0 0"/>
+    </joint>
+    <joint name="front_right_wheel_to_leg" type="continuous">
+        <parent link="front_right_leg"/>
+        <child link="front_right_wheel"/>
+        <origin xyz="-0.0925 -0.387904 -0.009518" rpy="0 0 0"/>
+        <axis xyz="1 0 0"/>
+    </joint>
+    <joint name="back_left_wheel_to_leg" type="continuous">
+        <parent link="back_left_leg"/>
+        <child link="back_left_wheel"/>
+        <origin xyz="0.0925 0.387904 -0.009518" rpy="0 0 0"/>
+        <axis xyz="1 0 0"/>
+    </joint>
+    <joint name="back_right_wheel_to_leg" type="continuous">
+        <parent link="back_right_leg"/>
+        <child link="back_right_wheel"/>
+        <origin xyz="-0.0925 0.387904 -0.009518" rpy="0 0 0"/>
         <axis xyz="1 0 0"/>
     </joint>

Commit message: simplified geometry

File: src/mks_description/urdf/eve.urdf.xacro (robot description, xacro)
@@ -1,10 +1,11 @@
 <?xml version="1.0"?>
 <robot xmlns:xacro="http://www.ros.org/wiki/xacro"  name="eve">
-    <link name="world" />
+    <xacro:arg name="mesh_path" default="package://mks_description/meshes"/>
+    <!-- <link name="world" /> -->
     <link name="chassis">
         <visual>
             <origin xyz="0 0 0.0" rpy="${pi/2} 0 0"/>
             <geometry>
-                <mesh filename="package://mks_description/meshes/chassis.stl" scale="0.001 0.001 0.001"/>
+                <mesh filename="$(arg mesh_path)/chassis.stl" scale="0.001 0.001 0.001"/>
             </geometry>
         </visual>
@@ -12,5 +13,5 @@
             <origin xyz="0 0 0" rpy="${pi/2} 0 0"/>
             <geometry>
-                <mesh filename="package://mks_description/meshes/chassis.stl" scale="0.001 0.001 0.001"/>
+                <mesh filename="$(arg mesh_path)/simplified_meshes/chassis_simp.stl" scale="0.001 0.001 0.001"/>
             </geometry>
         </collision>
@@ -18,17 +19,17 @@
             <origin xyz="0 0 0" rpy="0 0 0"/>
             <mass value="5.0"/>
-            <inertia ixx="0.2" ixy="0" ixz="0" iyy="0.3" iyz="0" izz="0.1"/>
-        </inertial>
-    </link>
-    <joint name="base_joint" type="fixed">
+            <inertia ixx="0.013" ixy="0" ixz="0" iyy="0.009" iyz="0" izz="0.005"/>
+        </inertial>
+    </link>
+    <!-- <joint name="base_joint" type="fixed">
         <parent link="world"/>
         <child link="chassis"/>
         <origin xyz="0 0 0" rpy="0 0 0"/>
-    </joint>
+    </joint> -->
     <link name="front_left_leg">
         <visual>
             <origin xyz="-0.247 0.058093 -0.025691" rpy="${pi/2} 0 0"/>
             <geometry>
-                <mesh filename="package://mks_description/meshes/front_left_leg.stl" scale="0.001 0.001 0.001"/>
+                <mesh filename="$(arg mesh_path)/front_left_leg.stl" scale="0.001 0.001 0.001"/>
             </geometry>
         </visual>
@@ -36,11 +37,11 @@
             <origin xyz="-0.247 0.058093 -0.025691" rpy="${pi/2} 0 0"/>
             <geometry>
-                <mesh filename="package://mks_description/meshes/front_left_leg.stl" scale="0.001 0.001 0.001"/>
-            </geometry>
-        </collision>
-        <inertial>
-            <origin xyz="0 0 0" rpy="0 0 0"/>
-            <mass value="5.0"/>
-            <inertia ixx="0.2" ixy="0" ixz="0" iyy="0.3" iyz="0" izz="0.1"/>
+                <mesh filename="$(arg mesh_path)/simplified_meshes/front_left_leg_simp.stl" scale="0.001 0.001 0.001"/>
+            </geometry>
+        </collision>
+        <inertial>
+            <origin xyz="0 0 0" rpy="0 0 0"/>
+            <mass value="1.5"/>
+            <inertia ixx="0.008" ixy="0" ixz="0" iyy="0.008" iyz="0" izz="0.0009"/>
         </inertial>
     </link>
@@ -49,5 +50,5 @@
             <origin xyz="0.247 0.058093 -0.025691" rpy="${pi/2} 0 0"/>
             <geometry>
-                <mesh filename="package://mks_description/meshes/front_right_leg.stl" scale="0.001 0.001 0.001"/>
+                <mesh filename="$(arg mesh_path)/front_right_leg.stl" scale="0.001 0.001 0.001"/>
             </geometry>
         </visual>
@@ -55,11 +56,11 @@
             <origin xyz="0.247 0.058093 -0.025691" rpy="${pi/2} 0 0"/>
             <geometry>
-                <mesh filename="package://mks_description/meshes/front_right_leg.stl" scale="0.001 0.001 0.001"/>
-            </geometry>
-        </collision>
-        <inertial>
-            <origin xyz="0 0 0" rpy="0 0 0"/>
-            <mass value="5.0"/>
-            <inertia ixx="0.2" ixy="0" ixz="0" iyy="0.3" iyz="0" izz="0.1"/>
+                <mesh filename="$(arg mesh_path)/simplified_meshes/front_right_leg_simp.stl" scale="0.001 0.001 0.001"/>
+            </geometry>
+        </collision>
+        <inertial>
+            <origin xyz="0 0 0" rpy="0 0 0"/>
+            <mass value="1.5"/>
+            <inertia ixx="0.008" ixy="0" ixz="0" iyy="0.008" iyz="0" izz="0.0009"/>
         </inertial>
     </link>
@@ -68,5 +69,5 @@
             <origin xyz="-0.247 -0.058093 -0.025691" rpy="${pi/2} 0 0"/>
             <geometry>
-                <mesh filename="package://mks_description/meshes/back_left_leg.stl" scale="0.001 0.001 0.001"/>
+                <mesh filename="$(arg mesh_path)/back_left_leg.stl" scale="0.001 0.001 0.001"/>
             </geometry>
         </visual>
@@ -74,11 +75,11 @@
             <origin xyz="-0.247 -0.058093 -0.025691" rpy="${pi/2} 0 0"/>
             <geometry>
-                <mesh filename="package://mks_description/meshes/back_left_leg.stl" scale="0.001 0.001 0.001"/>
-            </geometry>
-        </collision>
-        <inertial>
-            <origin xyz="0 0 0" rpy="0 0 0"/>
-            <mass value="5.0"/>
-            <inertia ixx="0.2" ixy="0" ixz="0" iyy="0.3" iyz="0" izz="0.1"/>
+                <mesh filename="$(arg mesh_path)/simplified_meshes/back_left_leg_simp.stl" scale="0.001 0.001 0.001"/>
+            </geometry>
+        </collision>
+        <inertial>
+            <origin xyz="0 0 0" rpy="0 0 0"/>
+            <mass value="1.5"/>
+            <inertia ixx="0.008" ixy="0" ixz="0" iyy="0.008" iyz="0" izz="0.0009"/>
         </inertial>
     </link>
@@ -87,5 +88,5 @@
             <origin xyz="0.247 -0.058093 -0.025691" rpy="${pi/2} 0 0"/>
             <geometry>
-                <mesh filename="package://mks_description/meshes/back_right_leg.stl" scale="0.001 0.001 0.001"/>
+                <mesh filename="$(arg mesh_path)/back_right_leg.stl" scale="0.001 0.001 0.001"/>
             </geometry>
         </visual>
@@ -93,11 +94,11 @@
             <origin xyz="0.247 -0.058093 -0.025691" rpy="${pi/2} 0 0"/>
             <geometry>
-                <mesh filename="package://mks_description/meshes/back_right_leg.stl" scale="0.001 0.001 0.001"/>
-            </geometry>
-        </collision>
-        <inertial>
-            <origin xyz="0 0 0" rpy="0 0 0"/>
-            <mass value="5.0"/>
-            <inertia ixx="0.2" ixy="0" ixz="0" iyy="0.3" iyz="0" izz="0.1"/>
+                <mesh filename="$(arg mesh_path)/simplified_meshes/back_right_leg_simp.stl" scale="0.001 0.001 0.001"/>
+            </geometry>
+        </collision>
+        <inertial>
+            <origin xyz="0 0 0" rpy="0 0 0"/>
+            <mass value="1.5"/>
+            <inertia ixx="0.008" ixy="0" ixz="0" iyy="0.008" iyz="0" izz="0.0009"/>
         </inertial>
     </link>
@@ -106,17 +107,17 @@
             <origin xyz="-0.3395 0.445997 -0.016173" rpy="${pi/2} 0 0"/>
             <geometry>
-                <mesh filename="package://mks_description/meshes/front_left_wheel.stl" scale="0.001 0.001 0.001"/>
-            </geometry>
-        </visual>
-        <collision>
-            <origin xyz="-0.3395 0.445997 -0.016173" rpy="${pi/2} 0 0"/>
-            <geometry>
-                <mesh filename="package://mks_description/meshes/front_left_wheel.stl" scale="0.001 0.001 0.001"/>
-            </geometry>
-        </collision>
-        <inertial>
-            <origin xyz="0 0 0" rpy="0 0 0"/>
-            <mass value="5.0"/>
-            <inertia ixx="0.2" ixy="0" ixz="0" iyy="0.3" iyz="0" izz="0.1"/>
+                <mesh filename="$(arg mesh_path)/front_left_wheel.stl" scale="0.001 0.001 0.001"/>
+            </geometry>
+        </visual>
+        <collision>
+            <origin xyz="-0.3395 0.445997 -0.016173" rpy="${pi/2} 0 0"/>
+            <geometry>
+                <mesh filename="$(arg mesh_path)/simplified_meshes/front_left_wheel_simp.stl" scale="0.001 0.001 0.001"/>
+            </geometry>
+        </collision>
+        <inertial>
+            <origin xyz="0 0 0" rpy="0 0 0"/>
+            <mass value="0.8"/>
+            <inertia ixx="0.001" ixy="0" ixz="0" iyy="0.0009" iyz="0" izz="0.0009"/>
         </inertial>
     </link>
@@ -125,17 +126,17 @@
             <origin xyz="0.3395 0.445997 -0.016173" rpy="${pi/2} 0 0"/>
             <geometry>
-                <mesh filename="package://mks_description/meshes/front_right_wheel.stl" scale="0.001 0.001 0.001"/>
-            </geometry>
-        </visual>
-        <collision>
-            <origin xyz="0.3395 0.445997 -0.016173" rpy="${pi/2} 0 0"/>
-            <geometry>
-                <mesh filename="package://mks_description/meshes/front_right_wheel.stl" scale="0.001 0.001 0.001"/>
-            </geometry>
-        </collision>
-        <inertial>
-            <origin xyz="0 0 0" rpy="0 0 0"/>
-            <mass value="5.0"/>
-            <inertia ixx="0.2" ixy="0" ixz="0" iyy="0.3" iyz="0" izz="0.1"/>
+                <mesh filename="$(arg mesh_path)/front_right_wheel.stl" scale="0.001 0.001 0.001"/>
+            </geometry>
+        </visual>
+        <collision>
+            <origin xyz="0.3395 0.445997 -0.016173" rpy="${pi/2} 0 0"/>
+            <geometry>
+                <mesh filename="$(arg mesh_path)/simplified_meshes/front_right_wheel_simp.stl" scale="0.001 0.001 0.001"/>
+            </geometry>
+        </collision>
+        <inertial>
+            <origin xyz="0 0 0" rpy="0 0 0"/>
+            <mass value="0.8"/>
+            <inertia ixx="0.001" ixy="0" ixz="0" iyy="0.0009" iyz="0" izz="0.0009"/>
         </inertial>
     </link>
@@ -144,17 +145,17 @@
             <origin xyz="-0.3395 0.445997 -0.016173" rpy="${pi/2} 0 0"/>
             <geometry>
-                <mesh filename="package://mks_description/meshes/back_left_wheel.stl" scale="0.001 0.001 0.001"/>
-            </geometry>
-        </visual>
-        <collision>
-            <origin xyz="-0.3395 0.445997 -0.016173" rpy="${pi/2} 0 0"/>
-            <geometry>
-                <mesh filename="package://mks_description/meshes/back_left_wheel.stl" scale="0.001 0.001 0.001"/>
-            </geometry>
-        </collision>
-        <inertial>
-            <origin xyz="0 0 0" rpy="0 0 0"/>
-            <mass value="5.0"/>
-            <inertia ixx="0.2" ixy="0" ixz="0" iyy="0.3" iyz="0" izz="0.1"/>
+                <mesh filename="$(arg mesh_path)/back_left_wheel.stl" scale="0.001 0.001 0.001"/>
+            </geometry>
+        </visual>
+        <collision>
+            <origin xyz="-0.3395 0.445997 -0.016173" rpy="${pi/2} 0 0"/>
+            <geometry>
+                <mesh filename="$(arg mesh_path)/simplified_meshes/back_left_wheel_simp.stl" scale="0.001 0.001 0.001"/>
+            </geometry>
+        </collision>
+        <inertial>
+            <origin xyz="0 0 0" rpy="0 0 0"/>
+            <mass value="0.8"/>
+            <inertia ixx="0.001" ixy="0" ixz="0" iyy="0.0009" iyz="0" izz="0.0009"/>
         </inertial>
     </link>
@@ -163,17 +164,17 @@
             <origin xyz="0.3395 0.445997 -0.016173" rpy="${pi/2} 0 0"/>
             <geometry>
-                <mesh filename="package://mks_description/meshes/back_right_wheel.stl" scale="0.001 0.001 0.001"/>
-            </geometry>
-        </visual>
-        <collision>
-            <origin xyz="0.3395 0.445997 -0.016173" rpy="${pi/2} 0 0"/>
-            <geometry>
-                <mesh filename="package://mks_description/meshes/back_right_wheel.stl" scale="0.001 0.001 0.001"/>
-            </geometry>
-        </collision>
-        <inertial>
-            <origin xyz="0 0 0" rpy="0 0 0"/>
-            <mass value="5.0"/>
-            <inertia ixx="0.2" ixy="0" ixz="0" iyy="0.3" iyz="0" izz="0.1"/>
+                <mesh filename="$(arg mesh_path)/back_right_wheel.stl" scale="0.001 0.001 0.001"/>
+            </geometry>
+        </visual>
+        <collision>
+            <origin xyz="0.3395 0.445997 -0.016173" rpy="${pi/2} 0 0"/>
+            <geometry>
+                <mesh filename="$(arg mesh_path)/simplified_meshes/back_right_wheel_simp.stl" scale="0.001 0.001 0.001"/>
+            </geometry>
+        </collision>
+        <inertial>
+            <origin xyz="0 0 0" rpy="0 0 0"/>
+            <mass value="0.8"/>
+            <inertia ixx="0.001" ixy="0" ixz="0" iyy="0.0009" iyz="0" izz="0.0009"/>
         </inertial>
     </link>
