Commit message: added world file

File: src/mks_description/urdf/eve.urdf.xacro (robot description, xacro)
@@ -2,5 +2,5 @@
 <robot xmlns:xacro="http://www.ros.org/wiki/xacro"  name="eve">
     <xacro:arg name="mesh_path" default="package://mks_description/meshes"/>
-    <!-- <link name="world" /> -->
+    <link name="root" />
     <link name="chassis">
         <visual>
@@ -22,9 +22,9 @@
         </inertial>
     </link>
-    <!-- <joint name="base_joint" type="fixed">
-        <parent link="world"/>
+    <joint name="base_joint" type="fixed">
+        <parent link="root"/>
         <child link="chassis"/>
         <origin xyz="0 0 0" rpy="0 0 0"/>
-    </joint> -->
+    </joint>
     <link name="front_left_leg">
         <visual>

Commit message: minor changes

File: src/mks_description/urdf/eve.urdf.xacro (robot description, xacro)
@@ -232,3 +232,21 @@
         <axis xyz="1 0 0"/>
     </joint>
+    <ros2_control name="GazeboSimSystem" type="system">
+        <hardware>
+        <plugin>gz_ros2_control/GazeboSimSystem</plugin>
+        </hardware>
+        <joint name="front_left_wheel_to_leg">
+        <command_interface name="velocity">
+            <param name="min">-1</param>
+            <param name="max">1</param>
+        </command_interface>
+        <state_interface name="position"/>
+        <state_interface name="velocity"/>
+        </joint>
+    </ros2_control>
+    <gazebo>
+        <plugin filename="gz_ros2_control-system" name="gz_ros2_control::GazeboSimROS2ControlPlugin">
+            <parameters>$(find mks_description)/config/eve_controller.yaml</parameters>
+        </plugin>
+    </gazebo>
 </robot>
